File: PROYECTO_KICAD/PROYECTO_KICAD.kicad_pcb (KiCad board)
At the start: 2 copper layers, 21 parts, among them J1 Conn_01x08_Pin, U1 NRF24L01, Y1 Crystal

Commit message: tarea
Parts:
- moved AE1 2.86 mm to (142.8, 75.8)
- moved J1 1.06 mm to (154.2, 87.5)
- moved C11 0.12 mm to (140.1, 78.4)
- moved R2 0.10 mm to (158.6, 82.4)
- moved C10 0.06 mm to (143.2, 78.4)
- moved C9 0.05 mm to (144.3, 78.4)
Connections:
- C1 pad 1: VDD -> GND
- C3 pad 1: VDD -> GND
- J1 pad 1: VDD -> GND
- U1 pad 15: VDD -> GND
- U1 pad 18: VDD -> GND
- U1 pad 21: (no net) -> GND
- U1 pad 7: VDD -> GND
Routing:
- net GND: track 0.00 -> 20.9 mm, vias 0 -> 7
- net Net-(J1-Pin_7): track 0.00 -> 7.70 mm, vias 0 -> 1
- net Net-(U1-XC2): track 0.00 -> 7.40 mm
- net Net-(U1-VDD_PA): track 0.00 -> 7.19 mm, vias 0 -> 2
- net Net-(U1-XC1): track 0.00 -> 7.11 mm
- net Net-(U1-ANT1): track 0.00 -> 4.77 mm
- net Net-(AE1-A): track 0.00 -> 3.90 mm
- net Net-(J1-Pin_2): track 0.00 -> 3.58 mm
- net Net-(J1-Pin_3): track 0.00 -> 3.56 mm, vias 0 -> 1
- net Net-(U1-ANT2): track 0.00 -> 3.39 mm
- net Net-(J1-Pin_6): track 0.00 -> 3.34 mm
- net Net-(C10-Pad1): track 0.00 -> 3.32 mm
- net Net-(J1-Pin_5): track 0.00 -> 3.03 mm
- net Net-(J1-Pin_4): track 0.00 -> 2.75 mm
- net Net-(U1-DVDD): track 0.00 -> 1.80 mm
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- added copper zone on B.Cu, net GND
- added copper zone on F.Cu, net GND
Other:
- board outline added: 20.5 x 20.3 mm
