File: PROYECTOS_KICAD/AISLADOR/aislador/aislador.kicad_sch (KiCad schematic)
At the start: 20 parts, among them IC1 ADUM3165BRSZ-RL, J1 USB_C_Receptacle_USB2.0_16P, J10 Conn_01x04_Pin, J2 USB_A, J3 Screw_Terminal_01x02, J4 Conn_01x03_Pin, J5 Conn_01x02_Pin, J6 Screw_Terminal_01x02, J7 Conn_01x02_Pin, J8 Conn_01x03_Pin, J9 Conn_01x03_Pin, Y1 LFXTAL071257Reel

Commit message: aislador_3160
Parts:
- removed C1: 10μF, symbol Device:C
- added C10, C7: 0.1μF, Capacitor_SMD:C_0402_1005Metric, symbol Device:C
- added C6: 0.1μF, Capacitor_SMD:C_0805_2012Metric, symbol Device:C
- added C8: 10μF, Capacitor_SMD:C_0805_2012Metric, symbol Device:C
- added J11, J12, J13: Conn_01x02_Pin, Connector_PinHeader_2.54mm:PinHeader_1x02_P2.54mm_Vertical, symbol Connector:Conn_01x02_Pin
- added J14, J16: Conn_01x03_Pin, Connector_PinHeader_2.54mm:PinHeader_1x03_P2.54mm_Vertical, symbol Connector:Conn_01x03_Pin
- added J15: Conn_01x04_Pin, Connector_PinHeader_2.54mm:PinHeader_1x04_P2.54mm_Vertical, symbol Connector:Conn_01x04_Pin
- C2, C3: footprint (none) -> Capacitor_SMD:C_0402_1005Metric
- C4, C5: value C -> 8pF; footprint (none) -> Capacitor_SMD:C_0402_1005Metric
- J10: footprint (none) -> Connector_PinHeader_2.54mm:PinHeader_1x04_P2.54mm_Vertical
- R1: footprint (none) -> Resistor_SMD:R_0603_1608Metric
Connections:
- net GND1: now also J1.S1 (SHIELD), C8.2; no longer IC1.5 (XI1)
- net Y1_-: now reaches C5.1, IC1.6 (XO1), Y1.3 (CRYSTAL_2)
- net at C2.1, IC1.1 (VBUS1), J4.2 (Pin_2)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: now also C8.1
- net Y1_+: now reaches C4.1, Y1.1 (CRYSTAL_1)
- net Y1_+: now also IC1.5 (XI1)
- net VBUS2: now reaches J6.1 (Pin_1)
- net VBUS2: now also IC1.20 (VBUS2), C6.1, C7.1, J11.2 (Pin_2), J12.2 (Pin_2)
- net GND2: now reaches J6.2 (Pin_2)
- net GND2: now also D2.2 (COMMON_A_1), D2.5 (COMMON_A_2), IC1.11 (GND2_1), IC1.15 (GND2_2), IC1.16 (GND2_3), IC1.17 (GND2_4), IC1.19 (GND2_5), J2.4 (GND), J2.5 (Shield), C10.2, C6.2, C7.2, J14.2 (Pin_2), J14.3 (Pin_3), J15.1 (Pin_1), J15.4 (Pin_4), J16.2 (Pin_2), J16.3 (Pin_3)
- net DD+: now reaches IC1.12 (DD+)
- net DD+: now also D2.1 (K_1), J2.3 (D+), J15.2 (Pin_2)
- net DD-: now reaches IC1.13 (DD-)
- net DD-: now also D2.3 (K_2), J2.2 (D-), J15.3 (Pin_3)
- net PGOOD: now reaches IC1.14 (PGOOD)
- net PGOOD: now also J16.1 (Pin_1)
- net at IC1.18 (VDD2): now also C10.1, J13.2 (Pin_2), J14.1 (Pin_1)
- net at J1.A5 (CC1), R1.1: now also J1.B5 (CC2)
- net VBUSOUT: now reaches J2.1 (VBUS)
- net VBUSOUT: now also J11.1 (Pin_1)
- net D+ renamed UD+
- net D- renamed UD-
Other:
- moved on the sheet: D2, J2, J3, J5, J6
