File: PROYECTOS_KICAD/AISLADOR_3160/AISLADOR_3160.kicad_pcb (KiCad board)
At the start: 2 copper layers, 51.8 x 20.8 mm, 21 parts, among them IC1 ADUM3160BRWZ, J1 USB_B, J2 USB_A, U1 TME-0505S, U2 USBLC6-2SC6, U3 USBLC6-2SC6

Commit message: aislador
Parts:
- added C7: C, Capacitor_SMD:C_2220_5750Metric, F.Cu at (147.3, 97.2)
Routing:
- net GND2: vias 261 -> 276
- net GND1: vias 265 -> 269

Commit message: aislador
Parts:
- added C8: C, Capacitor_SMD:CP_Elec_5x5.4, F.Cu at (175.8, 95.0)
- added D1: LED, LED_SMD:LED_0402_1005Metric, F.Cu at (143.2, 97.8)
- added R1: R, Resistor_SMD:R_0402_1005Metric, F.Cu at (143.2, 96.1)
- C7: footprint Capacitor_SMD:C_2220_5750Metric -> Capacitor_SMD:CP_Elec_5x5.4
Connections:
- J1 pad 5: unconnected-(J1-Shield-Pad5) -> GND1
Routing:
- net unconnected-(J1-Shield-Pad5): track 15.8 -> 0.00 mm
- net GND1: track 5.54 -> 21.4 mm, vias 269 -> 199
- net U2_+: track 4.01 -> 7.72 mm
- net +5V: track 45.0 -> 47.8 mm
- net VDD: track 27.3 -> 29.5 mm
- net Net-(D1-K): track 0.00 -> 1.72 mm
- net GND2: vias 276 -> 185
- added copper zone on B.Cu, net GND1
- added copper zone on B.Cu, net GND2

Commit message: ...
Routing:
- net GND2: vias 185 -> 152
- net GND1: vias 199 -> 120

Commit message: Avance
Routing:
- net GND2: track 12.9 -> 15.6 mm
- net GND1: track 21.4 -> 22.6 mm, vias 120 -> 121
